File: hardware/dual_pmod_vga/dual_pmod_vga.kicad_pcb (KiCad board)
At the start: 2 copper layers, 17 parts, among them J1 PMOD_1, J2 PMOD_2, J3 VGA_OUT

Commit message: minor fixes
Routing:
- net GND: track 151.7 -> 145.5 mm, vias 5 -> 4
- net Net-(J1-Pad8): track 12.5 -> 13.3 mm
- net Net-(J1-Pad4): track 9.77 -> 10.5 mm
- net Net-(J1-Pad6): track 11.1 -> 11.8 mm
- net Net-(J1-Pad7): track 23.4 -> 24.1 mm
- net Net-(J1-Pad1): track 10.3 -> 10.9 mm
